Commit message: 19July24

File: jupiter/description/4wd.urdf.xacro (robot description, xacro)
@@ -6,6 +6,6 @@
   <xacro:include filename="$(find jupiter)/description/skid_steer.urdf.xacro" />
   <xacro:include filename="$(find jupiter)/sensors/imu.urdf.xacro" />
-  <xacro:include filename="$(find jupiter)/sensors/generic_laser.urdf.xacro" />
-  <xacro:include filename="$(find jupiter)/sensors/depth_sensor.urdf.xacro" />
+  <xacro:include filename="$(find jupiter)/sensors/ldlidar.urdf.xacro" />
+  <xacro:include filename="$(find jupiter)/sensors/camera.urdf.xacro" />
   <xacro:base
     length="${base_length}"
@@ -53,10 +53,12 @@
   />
   <xacro:imu/>
-  <xacro:generic_laser>
+  <xacro:ldlidar/>
+  <xacro:camera/>
+  <!-- <xacro:generic_laser>
     <xacro:insert_block name="laser_pose" />
   </xacro:generic_laser>
   <xacro:depth_sensor>
     <xacro:insert_block name="depth_sensor_pose" />
-  </xacro:depth_sensor>
+  </xacro:depth_sensor> -->
   <xacro:diff_drive_controller
     wheel_separation="${wheel_pos_y * 2}"

File: jupiter/description/4wd_properties.urdf.xacro (robot description, xacro)
@@ -12,9 +12,8 @@
   <xacro:property name="wheel_mass" value=".150" />
   <xacro:property name="wheel_torque" value="20" />
+  <xacro:property name="usb_lidar" value="/dev/ttyUSB1" />
+  <xacro:property name="usb_mcu" value="/dev/ttyUSB0" />
   <xacro:property name="laser_pose">
     <origin xyz="0.060 0 0.145" rpy="0 0 0"/>
   </xacro:property>
-  <xacro:property name="depth_sensor_pose">
-    <origin xyz="0.080 0 0.020" rpy="0 0 0"/>
-  </xacro:property>
 </robot>

File: jupiter/sensors/camera.urdf.xacro (robot description, xacro)
@@ -1,10 +1,10 @@
 <robot xmlns:xacro="http://ros.org/wiki/xacro">
   <xacro:property name="M_PI" value="3.1415926535897931" />
-  <xacro:macro name="depth_sensor" params="*origin">
+  <xacro:macro name="camera">
     <link name="camera_link">
       <visual>
         <origin xyz="0 0 0" rpy="0 0 0"/>
         <geometry>
-          <box size="0.030 0.124 0.030"/>
+          <box size="0.020 0.095 0.050"/>
           <!-- <mesh filename="" scale="0.001 0.001 0.001"/> -->
         </geometry>
@@ -16,5 +16,5 @@
         <origin xyz="0 0 0" rpy="0 0 0"/>
         <geometry>
-          <box size="0.030 0.124 0.030"/>
+          <box size="0.020 0.095 0.050"/>
         </geometry>
       </collision>
@@ -27,4 +27,9 @@
       </inertial>
     </link>
+    <joint name="camera_to_base_link" type="fixed">
+      <parent link="base_link"/>
+      <child link="camera_link"/>
+      <origin xyz="0.120 0 0.020" rpy="0 0 0"/>
+    </joint>
     <gazebo reference="camera_link">
       <visual>
@@ -37,15 +42,4 @@
       </visual>
     </gazebo>
-    <joint name="camera_to_base_link" type="fixed">
-      <parent link="base_link"/>
-      <child link="camera_link"/>
-      <xacro:insert_block name="origin" />
-    </joint>
-    <link name="camera_depth_link"/>
-    <joint name="camera_depth_joint" type="fixed">
-      <origin xyz="0 0 0" rpy="-1.57 0 -1.57"/>
-      <parent link="camera_link"/>
-      <child link="camera_depth_link"/>
-    </joint>
     <!-- https://github.com/ros-simulation/gazebo_ros_pkgs/wiki/ROS-2-Migration:-Camera#gazebo_ros_camera -->
     <gazebo reference="camera_link">

File: jupiter/sensors/generic_laser.urdf.xacro (robot description, xacro)
@@ -4,11 +4,11 @@
   <xacro:macro name="generic_laser" params="*origin">
     <xacro:laser
-      update_rate="10"
+      update_rate="8"
       ray_count="360"
       min_angle="-3.1416"
       max_angle="3.1416"
       min_range="0.08"
-      max_range="12.0"
-      frame_id="laser"
+      max_range="8.0"
+      frame_id="laser_link"
       topic_name="scan"
     >
@@ -16,17 +16,3 @@
     </xacro:laser>
   </xacro:macro>
-  <xacro:macro name="generic_base_laser" params="*origin">
-    <xacro:laser
-      update_rate="10"
-      ray_count="360"
-      min_angle="-3.1416"
-      max_angle="3.1416"
-      min_range="0.21"
-      max_range="5.5"
-      frame_id="base_laser"
-      topic_name="base/scan"
-    >
-      <xacro:insert_block name="origin" />
-    </xacro:laser>
-  </xacro:macro>
 </robot>

File: jupiter/sensors/imu.urdf.xacro (robot description, xacro)
@@ -1,9 +1,20 @@
 <robot xmlns:xacro="http://ros.org/wiki/xacro">
   <xacro:macro name="imu">
-    <link name="imu_link"/>
+    <link name="imu_link">
+      <visual>
+        <origin xyz="0 0 0" rpy="0 0 0"/>
+        <geometry>
+          <box size="0.030 0.020 0.005"/>
+          <!-- <mesh filename="" scale="0.001 0.001 0.001"/> -->
+        </geometry>
+        <material name="red">
+          <color rgba="0.416 0.051 0.047 1.0"/>
+        </material>
+      </visual>
+    </link>
     <joint name="imu_to_base_link" type="fixed">
       <parent link="base_link"/>
       <child link="imu_link"/>
-      <origin xyz="0.130 0 0.015" rpy="0 0 0"/>
+      <origin xyz="0.015 0 0.070" rpy="0 0 0"/>
     </joint>
     <gazebo reference="imu_link">
