Commit message: 20july24 update

File: jupiter/description/jupiter.urdf.xacro (robot description, xacro)
@@ -1,5 +1,5 @@
 <?xml version="1.0"?>
 <robot name="jupiter" xmlns:xacro="http://ros.org/wiki/xacro">
-  <xacro:include filename="$(find jupiter)/description/4wd_properties.urdf.xacro" />
+  <xacro:include filename="$(find jupiter)/description/jupiter_properties.urdf.xacro" />
   <xacro:include filename="$(find jupiter)/description/base.urdf.xacro" />
   <xacro:include filename="$(find jupiter)/description/wheel.urdf.xacro" />
@@ -55,10 +55,4 @@
   <xacro:ldlidar/>
   <xacro:camera/>
-  <!-- <xacro:generic_laser>
-    <xacro:insert_block name="laser_pose" />
-  </xacro:generic_laser>
-  <xacro:depth_sensor>
-    <xacro:insert_block name="depth_sensor_pose" />
-  </xacro:depth_sensor> -->
   <xacro:diff_drive_controller
     wheel_separation="${wheel_pos_y * 2}"

File: jupiter/description/jupiter_properties.urdf.xacro (robot description, xacro)
@@ -1,3 +1,4 @@
 <?xml version="1.0"?>
+<!-- jupiter robot property settings - change the robot dimensions and wheel properties HERE -->
 <robot xmlns:xacro="http://ros.org/wiki/xacro">
   <xacro:property name="base_length" value="0.305" />
@@ -14,6 +15,3 @@
   <xacro:property name="usb_lidar" value="/dev/ttyUSB1" />
   <xacro:property name="usb_mcu" value="/dev/ttyUSB0" />
-  <xacro:property name="laser_pose">
-    <origin xyz="0.060 0 0.145" rpy="0 0 0"/>
-  </xacro:property>
 </robot>
