Commit message: urdf updates

File: jupiter/description/base.urdf.xacro (robot description, xacro)
@@ -7,4 +7,5 @@
       <child link="base_link"/>
       <origin xyz="0 0 ${wheel_radius - wheel_pos_z}" rpy="0 0 0"/>
+      <!-- <origin xyz="0 0 0" rpy="0 0 0"/> -->
     </joint>
     <link name="base_link">

File: jupiter/description/jupiter_properties.urdf.xacro (robot description, xacro)
@@ -8,7 +8,7 @@
   <xacro:property name="wheel_radius" value="0.045" />
   <xacro:property name="wheel_width" value="0.045" />
-  <xacro:property name="wheel_pos_x" value="0.087" />
+  <xacro:property name="wheel_pos_x" value="0.090" />
   <xacro:property name="wheel_pos_y" value="0.175" />
-  <xacro:property name="wheel_pos_z" value="-0.034" />
+  <xacro:property name="wheel_pos_z" value="-0.035" />  <!-- wheel_z_pos = 1/2 x base_height - wheel_radius -->
   <xacro:property name="wheel_mass" value=".150" />
   <xacro:property name="wheel_torque" value="20" />

File: jupiter/description/wheel.urdf.xacro (robot description, xacro)
@@ -26,4 +26,10 @@
       </inertial>
     </link>
+    <joint name="${side}_wheel_joint" type="continuous">
+      <axis xyz="0 1 0" />
+      <parent link="base_link"/>
+      <child link="${side}_wheel_link"/>
+      <origin xyz="${pos_x} ${pos_y} ${pos_z}" rpy="0 0 0"/>
+    </joint>
     <gazebo reference="${side}_wheel_link">
       <visual>
@@ -36,10 +42,4 @@
       </visual>
     </gazebo>
-    <joint name="${side}_wheel_joint" type="continuous">
-      <axis xyz="0 1 0" />
-      <parent link="base_link"/>
-      <child link="${side}_wheel_link"/>
-      <origin xyz="${pos_x} ${pos_y} ${pos_z}" rpy="0 0 0"/>
-    </joint>
   </xacro:macro>
 </robot>
