Commit message: update slam.yaml

File: jupiter/sensors/camera.urdf.xacro (robot description, xacro)
@@ -30,5 +30,5 @@
       <parent link="base_link"/>
       <child link="camera_link"/>
-      <origin xyz="0.120 0 0.020" rpy="0 0 0"/>
+      <origin xyz="0.115 0 0.130" rpy="0 0 0"/>
     </joint>
     <gazebo reference="camera_link">

File: jupiter/sensors/imu.urdf.xacro (robot description, xacro)
@@ -16,5 +16,5 @@
       <parent link="base_link"/>
       <child link="imu_link"/>
-      <origin xyz="0.015 0 0.070" rpy="0 0 0"/>
+      <origin xyz="0.020 0 0.070" rpy="0 0 0"/>
     </joint>
     <gazebo reference="imu_link">

File: jupiter/sensors/ldlidar.urdf.xacro (robot description, xacro)
@@ -15,5 +15,5 @@
       <parent link="base_link"/>
       <child link="laser_link"/>
-      <origin xyz="0.060 0 0.145" rpy="0 0 0"/>
+      <origin xyz="0.020 0 0.165" rpy="0 0 0"/>
     </joint>
     <gazebo reference="laser_link">
